File: KiCadFiles/TestBed_KL05_variant_01_f.kicad_pcb (KiCad board)
At the start: 2 copper layers, 100 x 100 mm, 30 parts, among them J1 CONN_ARDUINO_R3, J2 CONN_NUCLEO_MORPH

Commit message: Update PCB
Parts:
- added R23: 10 5W, Resistor_THT:R_Axial_DIN0411_L9.9mm_D3.6mm_P12.70mm_Horizontal, F.Cu at (133.3, 72.4)
Connections:
- J1 pad J1_2: /T_P3V3 -> /PA0
- J1 pad J1_4: /T_P3V3 -> /PA0
Routing:
- net /PA0: track 0.00 -> 127.5 mm
- net GND: vias 47 -> 51
- net (no net): vias 4 -> 0

Commit message: Dokumentacja
Parts:
- added JP7: Jumper, Connector_PinHeader_2.54mm:PinHeader_1x02_P2.54mm_Vertical, F.Cu at (132.1, 59.7)
- moved R23 6.35 mm to (127.0, 72.4)
Connections:
- R23 pad 2: /PA0 -> Net-(JP7-Pad1)
Routing:
- net Net-(JP7-Pad1): track 0.00 -> 5.08 mm
- net /PA0: track 127.5 -> 123.5 mm
