File: KiCadFiles/TestBed_KL05_variant_01_f.sch (KiCad schematic (older format))
At the start: 30 parts, among them J1 CONN_ARDUINO_R3, J2 CONN_NUCLEO_MORPH

Commit message: Update PCB
Parts:
- added R23: 10 5W, Resistor_THT:R_Axial_DIN0411_L9.9mm_D3.6mm_P12.70mm_Horizontal, symbol TestBed_KL05_variant_01_f-rescue:R_Small-Device
- JP1, JP2, JP3, JP4, JP5, JP6: symbol Device:Jumper_NC_Small -> TestBed_KL05_variant_01_f-rescue:Jumper_NC_Small-Device
- R1, R10, R11, R12, R13, R14, R15, R16, R17, R18, R19, R2, R20, R21, R22, R3, R4, R5, R6, R7, R8, R9: symbol Device:R_Small -> TestBed_KL05_variant_01_f-rescue:R_Small-Device
Connections:
- wire segments 149 -> 155
Other:
- note added: "CONFIGURATION SETUP FOR POWER SUPPLY TEST\n"
Changed lines of the file:
@@
 	3250 8200 3250 8100
 $Comp
-L Device:Jumper_NC_Small JP1
+L TestBed_KL05_variant_01_f-rescue:Jumper_NC_Small-Device JP1
 U 1 1 606F247C
 P 3550 7800
@@
 	3450 7800 3250 7800
 $Comp
-L Device:Jumper_NC_Small JP2
+L TestBed_KL05_variant_01_f-rescue:Jumper_NC_Small-Device JP2
 U 1 1 606F89B6
 P 3550 7900
@@
 $EndComp
 $Comp
-L Device:Jumper_NC_Small JP3
+L TestBed_KL05_variant_01_f-rescue:Jumper_NC_Small-Device JP3
 U 1 1 606F8BF6
 P 3550 8000
@@
 $EndComp
 $Comp
-L Device:Jumper_NC_Small JP4
+L TestBed_KL05_variant_01_f-rescue:Jumper_NC_Small-Device JP4
 U 1 1 606F8E45
 P 3550 8100
@@
 $EndComp
 $Comp
-L Device:Jumper_NC_Small JP5
+L TestBed_KL05_variant_01_f-rescue:Jumper_NC_Small-Device JP5
 U 1 1 606F9067
 P 3550 8200
@@
 $EndComp
 $Comp
-L Device:Jumper_NC_Small JP6
+L TestBed_KL05_variant_01_f-rescue:Jumper_NC_Small-Device JP6
 U 1 1 606F927F
 P 3550 8300
@@
 	8400 1750 7000 1750
 $Comp
-L Device:R_Small R1
+L TestBed_KL05_variant_01_f-rescue:R_Small-Device R1
 U 1 1 60F11522
 P 7900 2700
@@
 	7800 2700 7000 2700
 $Comp
-L Device:R_Small R2
+L TestBed_KL05_variant_01_f-rescue:R_Small-Device R2
 U 1 1 60F11FE1
 P 7900 2800
@@
 	7800 2800 7000 2800
 $Comp
-L Device:R_Small R3
+L TestBed_KL05_variant_01_f-rescue:R_Small-Device R3
 U 1 1 60F12134
 P 7900 2900
@@
 	7800 2900 7000 2900
 $Comp
-L Device:R_Small R4
+L TestBed_KL05_variant_01_f-rescue:R_Small-Device R4
 U 1 1 60F1221D
 P 7900 3000
@@
 	7800 3000 7000 3000
 $Comp
-L Device:R_Small R5
+L TestBed_KL05_variant_01_f-rescue:R_Small-Device R5
 U 1 1 60F12390
 P 7900 3100
@@
 	7800 3100 7000 3100
 $Comp
-L Device:R_Small R6
+L TestBed_KL05_variant_01_f-rescue:R_Small-Device R6
 U 1 1 60F1244F
 P 7900 3200
@@
 	7800 3200 7000 3200
 $Comp
-L Device:R_Small R15
+L TestBed_KL05_variant_01_f-rescue:R_Small-Device R15
 U 1 1 60F12647
 P 10600 2500
@@
 	10700 2500 11200 2500
 $Comp
-L Device:R_Small R16
+L TestBed_KL05_variant_01_f-rescue:R_Small-Device R16
 U 1 1 60F12DE3
 P 10600 2600
@@
 	10700 2600 11200 2600
 $Comp
-L Device:R_Small R17
+L TestBed_KL05_variant_01_f-rescue:R_Small-Device R17
 U 1 1 60F1319D
 P 10600 2700
@@
 	10700 2700 11200 2700
 $Comp
-L Device:R_Small R18
+L TestBed_KL05_variant_01_f-rescue:R_Small-Device R18
 U 1 1 60F13300
 P 10600 2800
@@
 	10700 2800 11200 2800
 $Comp
-L Device:R_Small R19
+L TestBed_KL05_variant_01_f-rescue:R_Small-Device R19
 U 1 1 60F13429
 P 10600 2900
@@
 	10700 2900 11200 2900
 $Comp
-L Device:R_Small R20
+L TestBed_KL05_variant_01_f-rescue:R_Small-Device R20
 U 1 1 60F1357B
 P 10600 3000
@@
 	10700 3000 11200 3000
 $Comp
-L Device:R_Small R21
+L TestBed_KL05_variant_01_f-rescue:R_Small-Device R21
 U 1 1 60F136ED
 P 10600 3100
@@
 	10700 3100 11200 3100
 $Comp
-L Device:R_Small R22
+L TestBed_KL05_variant_01_f-rescue:R_Small-Device R22
 U 1 1 60F1382B
 P 10600 3200
@@
 	10700 3200 11200 3200
 $Comp
-L Device:R_Small R7
+L TestBed_KL05_variant_01_f-rescue:R_Small-Device R7
 U 1 1 60F1395E
 P 10600 1450
@@
 	10500 1450 10000 1450
 $Comp
-L Device:R_Small R8
+L TestBed_KL05_variant_01_f-rescue:R_Small-Device R8
 U 1 1 60F13D06
 P 10600 1550
@@
 	10700 1550 11200 1550
 $Comp
-L Device:R_Small R9
+L TestBed_KL05_variant_01_f-rescue:R_Small-Device R9
 U 1 1 60F141AC
 P 10600 1850
@@
 	10700 1850 11200 1850
 $Comp
-L Device:R_Small R10
+L TestBed_KL05_variant_01_f-rescue:R_Small-Device R10
 U 1 1 60F144C4
 P 10600 1950
@@
 	10700 1950 11200 1950
 $Comp
-L Device:R_Small R11
+L TestBed_KL05_variant_01_f-rescue:R_Small-Device R11
 U 1 1 60F14636
 P 10600 2050
@@
 	10700 2050 11200 2050
 $Comp
-L Device:R_Small R12
+L TestBed_KL05_variant_01_f-rescue:R_Small-Device R12
 U 1 1 60F147E6
 P 10600 2150
@@
 	10700 2150 11200 2150
 $Comp
-L Device:R_Small R13
+L TestBed_KL05_variant_01_f-rescue:R_Small-Device R13
 U 1 1 60F14951
 P 10600 2250
@@
 	10700 2250 11200 2250
 $Comp
-L Device:R_Small R14
+L TestBed_KL05_variant_01_f-rescue:R_Small-Device R14
 U 1 1 60F14AB3
 P 10600 2350
@@
 	6300 3550 7550 3550
 $Comp
-L power:GND #PWR0101
+L TestBed_KL05_variant_01_f-rescue:GND-power #PWR0101
 U 1 1 6102BF9F
 P 5800 3150
@@
 NoConn ~ 5500 3400
 NoConn ~ 3300 2800
+$Comp
+L TestBed_KL05_variant_01_f-rescue:R_Small-Device R23
+U 1 1 612D32FB
+P 7500 8000
+F 0 "R23" V 7450 7750 50  0000 C CNN
+F 1 "10 5W" V 7395 8000 50  0000 C CNN
+F 2 "Resistor_THT:R_Axial_DIN0411_L9.9mm_D3.6mm_P12.70mm_Horizontal" H 7500 8000 50  0001 C CNN
+F 3 "~" H 7500 8000 50  0001 C CNN
+	1    7500 8000
+	0    1    1    0
+$EndComp
+Text Notes 6450 7650 0    50   ~ 10
+CONFIGURATION SETUP FOR POWER SUPPLY TEST\n
+Wire Wire Line
+	6800 8000 6800 7850
+Wire Wire Line
+	6800 8000 6800 8150
+Connection ~ 6800 8000
+Wire Wire Line
+	6800 7850 6500 7850
+Wire Wire Line
+	6800 8150 6500 8150
+Text Label 6500 8150 0    50   ~ 0
+PA0
+Text Label 8250 8000 2    50   ~ 0
+GND
+Text Label 6500 7850 0    50   ~ 0
+T_P3V3
+Wire Notes Line
+	8400 8600 6400 8600
+Wire Notes Line
+	6400 7550 6400 8600
+Wire Notes Line
+	8400 7550 8400 8600
+Wire Wire Line
+	6800 8000 7400 8000
+Wire Wire Line
+	7600 8000 8250 8000
 $EndSCHEMATC

Commit message: Dokumentacja
Parts:
- added JP7: Jumper, Connector_PinHeader_2.54mm:PinHeader_1x02_P2.54mm_Vertical, symbol TestBed_KL05_variant_01_f-rescue:Jumper_NC_Small-Device
Connections:
- net PA0: now also JP7.2; no longer R23.2
- new net: JP7.1, R23.2
Changed lines of the file:
@@
 	8400 7550 8400 8600
 Wire Wire Line
-	6800 8000 7400 8000
+	6800 8000 7000 8000
 Wire Wire Line
 	7600 8000 8250 8000
+$Comp
+L TestBed_KL05_variant_01_f-rescue:Jumper_NC_Small-Device JP7
+U 1 1 612DF240
+P 7100 8000
+F 0 "JP7" H 7250 8050 50  0000 C CNN
+F 1 "Jumper" H 7750 8050 50  0001 C CNN
+F 2 "Connector_PinHeader_2.54mm:PinHeader_1x02_P2.54mm_Vertical" H 7100 8000 50  0001 C CNN
+F 3 "~" H 7100 8000 50  0001 C CNN
+	1    7100 8000
+	-1   0    0    -1
+$EndComp
+Wire Wire Line
+	7200 8000 7400 8000
 $EndSCHEMATC
