File: KiCadFiles/TestBed_KL05_variant_02_f.kicad_pcb (KiCad board)
At the start: 2 copper layers, 100 x 100 mm, 51 parts, among them J1 CONN_ARDUINO_R3, J2 CONN_NUCLEO_MORPH, K1 RELAY, K2 RELAY, K3 RELAY, K4 RELAY, K5 RELAY, K6 RELAY, Q1 NMOS, Q2 NMOS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

Commit message: Dokumentacja
Parts:
- added JP1: , Connector_PinHeader_2.54mm:PinHeader_1x02_P2.54mm_Vertical, F.Cu at (134.6, 59.7)
- moved R29 6.35 mm to (127.0, 72.4)
Connections:
- R29 pad 2: /PA0 -> Net-(JP1-Pad2)
Routing:
- net Net-(JP1-Pad2): track 0.00 -> 5.08 mm
- net /PA0: track 137.0 -> 133.7 mm
- added copper zone on F.Cu, net GND
