File: KiCadFiles/TestBed_KL05_variant_02_f.sch (KiCad schematic (older format))
At the start: 50 parts, among them J1 CONN_ARDUINO_R3, J2 CONN_NUCLEO_MORPH, K1 RELAY, K2 RELAY, K3 RELAY, K4 RELAY, K5 RELAY, K6 RELAY, Q1 NMOS, Q2 NMOS, Q3 NMOS, Q4 NMOS, Q5 NMOS, Q6 NMOS

Commit message: Update PCB
Parts:
- added R29: 10 5W, Resistor_THT:R_Axial_DIN0411_L9.9mm_D3.6mm_P12.70mm_Horizontal, symbol TestBed_KL05_variant_02_f-rescue:R_Small-Device
- C1, C2: symbol Device:C_Small -> TestBed_KL05_variant_02_f-rescue:C_Small-Device
- D1, D2, D3, D4, D5, D6: symbol Device:D_Small -> TestBed_KL05_variant_02_f-rescue:D_Small-Device
- K1, K2, K3, K4, K5, K6: symbol Relay:UMS05-1A80-75L -> TestBed_KL05_variant_02_f-rescue:UMS05-1A80-75L-Relay
- Q1, Q2, Q3, Q4, Q5, Q6: symbol Device:Q_NMOS_DGS -> TestBed_KL05_variant_02_f-rescue:Q_NMOS_DGS-Device
- R1, R10, R11, R12, R13, R14, R15, R16, R17, R18, R19, R2, R20, R21, R22, R23, R24, R25, R26, R27, R28, R3, R4, R5, R6, R7, R8, R9: symbol Device:R_Small -> TestBed_KL05_variant_02_f-rescue:R_Small-Device
Connections:
- wire segments 223 -> 230
- no-connect marks 84 -> 82
Other:
- note added: "CONFIGURATION SETUP FOR POWER SUPPLY TEST"

Commit message: Dokumentacja
Parts:
- added JP1: (no value), Connector_PinHeader_2.54mm:PinHeader_1x02_P2.54mm_Vertical, symbol TestBed_KL05_variant_01_f-rescue:Jumper_NC_Small-Device
Connections:
- net PA0: now also JP1.1; no longer R29.2
- new net: JP1.2, R29.2
Other:
- moved on the sheet: R29
Changed lines of the file:
@@
 L TestBed_KL05_variant_02_f-rescue:R_Small-Device R29
 U 1 1 612DE971
-P 13450 8000
-F 0 "R29" V 13400 7750 50  0000 C CNN
-F 1 "10 5W" V 13345 8000 50  0000 C CNN
-F 2 "Resistor_THT:R_Axial_DIN0411_L9.9mm_D3.6mm_P12.70mm_Horizontal" H 13450 8000 50  0001 C CNN
-F 3 "~" H 13450 8000 50  0001 C CNN
-	1    13450 8000
+P 13650 8000
+F 0 "R29" V 13600 7750 50  0000 C CNN
+F 1 "10 5W" V 13545 8000 50  0000 C CNN
+F 2 "Resistor_THT:R_Axial_DIN0411_L9.9mm_D3.6mm_P12.70mm_Horizontal" H 13650 8000 50  0001 C CNN
+F 3 "~" H 13650 8000 50  0001 C CNN
+	1    13650 8000
 	0    1    1    0
 $EndComp
-Wire Wire Line
-	13350 8000 13000 8000
 Wire Wire Line
 	13000 8000 13000 7800
@@
 $EndComp
 Wire Wire Line
-	13550 8000 13900 8000
-Wire Wire Line
 	13900 8000 13900 8100
 Text Notes 12350 7300 0    50   ~ 10
@@
 Text Label 12700 7800 0    50   ~ 0
 T_P3V3
+$Comp
+L TestBed_KL05_variant_01_f-rescue:Jumper_NC_Small-Device JP1
+U 1 1 612E54C8
+P 13200 8000
+F 0 "JP1" H 13150 8100 50  0000 C CNN
+F 1 "  " H 13200 8121 50  0000 C CNN
+F 2 "Connector_PinHeader_2.54mm:PinHeader_1x02_P2.54mm_Vertical" H 13200 8000 50  0001 C CNN
+F 3 "" H 13200 8000 50  0001 C CNN
+	1    13200 8000
+	1    0    0    -1
+$EndComp
+Wire Wire Line
+	13100 8000 13000 8000
+Wire Wire Line
+	13900 8000 13750 8000
+Wire Wire Line
+	13300 8000 13550 8000
 $EndSCHEMATC
